File: ac-switcher.kicad_sch (KiCad schematic)
At the start: 25 parts, among them K1 Relay_SPDT, Q1 2N7000, Q2 2N7000, Q3 BT136-600, U3 10A SSR, U5 MOC3063S

Commit message: More mods
Parts:
- R12: renamed from R10; value 360R -> 360R 1W
- R14: renamed from R12; value 39R 1W -> 39R 2W
- R7: renamed from R9; value R so I=5mA -> R so I=10mA
- RV2: renamed from RV1; value Varistor -> Varistor 10D271K
- RV3: renamed from RV2; value Varistor -> Varistor 10D271K
- renumbered C1 to C3, C3 to C5, D1 to D3, F2 to F3, Q3 to Q2, Q2 to Q3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
