File: panoboard2.kicad_pcb (KiCad board)
At the start: 2 copper layers, 100 x 69.5 mm, 76 parts, among them J11 I2C1, J12 I2C2, J2 THERMISTOR, J6 BLK/MAINS L, J7 WHT/HTR, J8 ORA/MAINS N, J9 MOLEX 53375-0810, K1 Relay_SPDT, M2 TINYPICO, P2 PCB_Patch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

Commit message: Bumped version number
Other:
- board text added: "v1.0i 21-Jan-26"
- board text removed: "v1.0h 13-Jul-24"
Changed lines of the file:
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@@
 		)
 	)
-	(gr_text "v1.0h 13-Jul-24"
+	(gr_text "v1.0i 21-Jan-26"
 		(at 121.175 79.825 0)
 		(layer "F.SilkS")
